Commit message: feat: implemented two imu to mimic human arm (upper arm & Forearm)
Modified files:
- imu_tracker/imu_tracker/serial_bridge.py
- imu_tracker/setup.py
- imu_tracker/urdf/arm.urdf

File: imu_tracker/urdf/arm.urdf (robot description, URDF)
Before this commit: robot human_arm, 3 links, 2 joints
Joints:
- joint shoulder_joint: axis (none) -> 0 1 0; limit (none) -> lower=-1.57 upper=1.57 effort=1 velocity=1; type fixed -> revolute
